Commit message: urdf_updated

File: robot_description/models/robot_core.xacro (robot description, xacro)
@@ -1,5 +1,106 @@
 <?xml version="1.0"?>
 <robot xmlns:xacro = "http://www.ros.org/wiki/xacro" >
-    <link name="base_link">
+    <xacro:include filename="inertial_macros.xacro"/>
+    <!-- BASE LINK -->
+    <link name="base_link"></link>
+    <!-- CHASSIS LINK -->
+    <joint name="chassis_joint" type ="fixed">
+        <parent link="base_link"/>
+        <child link="chassis"/>
+        <origin xyz="-0.3 0.0 0.0"/>
+    </joint>
+    <link name="chassis">
+        <visual>
+            <origin xyz="0.2 0 0.075"/>
+            <geometry>
+                <box size="0.4 0.3 0.15"/>
+            </geometry>
+            <material name="gray">
+                <color rgba="0.5 0.5 0.5 1"/> <!-- Medium gray with full opacity -->
+            </material>
+        </visual>
+        <collision>
+            <origin xyz="0.2 0 0.075"/>
+            <geometry>
+                <box size="0.4 0.3 0.15"/>
+            </geometry>
+        </collision>
+        <xacro:inertial_box mass="2.9" x = "0.4" y="0.3" z="0.15">
+            <origin xyz="0.2 0 0.075" rpy="0 0 0"/>
+        </xacro:inertial_box>
+    </link>
+    <!-- LEFT WHEEL LINK -->
+    <joint name="left_wheel_joint" type="continuous">
+        <parent link="base_link"/>
+        <child link="left_wheel"/>
+        <origin xyz="0 0.16 0" rpy="-${pi/2} 0 0"/>
+        <axis xyz="0 0 1"/>
+    </joint>
+    <link name="left_wheel">
+        <visual>
+            <geometry>
+                <cylinder radius="0.05" length="0.02"/>
+            </geometry>
+            <material name="black">
+                <color rgba="0 0 0 1"/> <!-- black with full opacity -->
+            </material>
+        </visual>
+        <collision>
+            <geometry>
+                <cylinder radius="0.05" length="0.02"/>
+            </geometry>
+        </collision>
+        <xacro:inertial_cylinder mass="0.1" length="0.02" radius="0.05">
+            <origin xyz="0 0 0" rpy="0 0 0"/>
+        </xacro:inertial_cylinder>
+    </link>
+    <!-- RIGHT WHEEL LINK -->
+    <joint name="right_wheel_joint" type="continuous">
+        <parent link="base_link"/>
+        <child link="right_wheel"/>
+        <origin xyz="0 -0.16 0" rpy="${pi/2} 0 0"/>
+        <axis xyz="0 0 -1"/>
+    </joint>
+    <link name="right_wheel">
+        <visual>
+            <geometry>
+                <cylinder radius="0.05" length="0.02"/>
+            </geometry>
+            <material name="black">
+                <color rgba="0 0 0 1"/> <!-- black with full opacity -->
+            </material>
+        </visual>
+        <collision>
+            <geometry>
+                <cylinder radius="0.05" length="0.02"/>
+            </geometry>
+        </collision>
+        <xacro:inertial_cylinder mass="0.1" length="0.02" radius="0.05">
+            <origin xyz="0 0 0" rpy="0 0 0"/>
+        </xacro:inertial_cylinder>
+    </link>
+    <!-- CASTER WHEEL LINK -->
+    <joint name="caster_wheel_joint" type="fixed">
+        <parent link="chassis"/>
+        <child link="caster_wheel"/>
+        <origin xyz="0.05 0 0"/>
+    </joint>
+    <link name="caster_wheel">
+        <visual>
+            <geometry>
+                <sphere radius="0.05"/>
+            </geometry>
+            <material name="black">
+                <color rgba="0 0 0 1"/> <!-- black with full opacity -->
+            </material>
+        </visual>
+        <collision>
+            <geometry>
+                <sphere radius="0.05"/>
+            </geometry>
+        </collision>
+        <xacro:inertial_sphere mass="0.1" radius="0.05">
+            <origin xyz="0 0 0" rpy="0 0 0"/>
+        </xacro:inertial_sphere>
     </link>
 </robot>

Commit message: Added serial as a submodule

File: robot_description/models/robot_core.xacro (robot description, xacro)
@@ -17,5 +17,5 @@
             </geometry>
             <material name="gray">
-                <color rgba="0.5 0.5 0.5 1"/> <!-- Medium gray with full opacity -->
+                <color rgba="0.5 0.5 0.5 1"/>
             </material>
         </visual>
@@ -43,5 +43,5 @@
             </geometry>
             <material name="black">
-                <color rgba="0 0 0 1"/> <!-- black with full opacity -->
+                <color rgba="0 0 0 1"/>
             </material>
         </visual>
@@ -68,5 +68,5 @@
             </geometry>
             <material name="black">
-                <color rgba="0 0 0 1"/> <!-- black with full opacity -->
+                <color rgba="0 0 0 1"/>
             </material>
         </visual>
@@ -92,5 +92,5 @@
             </geometry>
             <material name="black">
-                <color rgba="0 0 0 1"/> <!-- black with full opacity -->
+                <color rgba="0 0 0 1"/>
             </material>
         </visual>
@@ -104,3 +104,29 @@
         </xacro:inertial_sphere>
     </link>
+        <!-- LiDAR -->
+    <joint name="lidar_joint" type="fixed">
+        <parent link="base_link"/>
+        <child link="lidar_link"/>
+        <origin xyz="0 0 0.17" rpy="0 0 0"/>
+    </joint>
+    <link name="lidar_link">
+        <visual>
+            <origin xyz="0 0 0" rpy="0 0 0"/>
+            <geometry>
+            <mesh filename="package://robot_description/meshes/YdlidarX2.stl" scale="0.001 0.001 0.001"/>
+            </geometry>
+            <material name="blue">
+                <color rgba="0 0 1 1"/>
+            </material>
+        </visual>
+        <collision>
+            <origin xyz="0 0 0" rpy="0 0 0"/>
+            <geometry>
+                <cylinder radius="0.05" length="0.03"/>
+            </geometry>
+        </collision>
+        <xacro:inertial_cylinder mass="0.2" radius="0.05" length="0.03">
+            <origin xyz="0 0 0" rpy="0 0 0"/>
+        </xacro:inertial_cylinder>
+    </link>
 </robot>

Commit message: update

File: robot_description/models/robot_core.xacro (robot description, xacro)
@@ -4,4 +4,9 @@
     <!-- BASE LINK -->
     <link name="base_link"></link>
+    <!-- <joint name="base_footprint" type="fixed">
+        <parent link="base_link"/>
+        <child link="base_footprint"/>
+        <origin xyz="0 0 0"/>
+    </joint> -->
     <!-- CHASSIS LINK -->
     <joint name="chassis_joint" type ="fixed">
